Commit message: Create gpu to enable/disable GPU processing

File: ca_description/urdf/roomblock.xacro (robot description, xacro)
@@ -8,5 +8,5 @@
   <xacro:include filename="$(find ca_description)/urdf/sensors/laser_sensor.xacro"/>
   <xacro:include filename="$(find ca_description)/urdf/sensors/camera_sensor.xacro"/>
-  <xacro:macro name="roomblock" params="parent visualize:=false">
+  <xacro:macro name="roomblock" params="parent visualize:=false gpu:=false">
     <xacro:property name="z" value="0.061"/>
     <xacro:property name="roomblock_link" value="block_link"/>
@@ -35,5 +35,5 @@
       </xacro:inertial_cuboid_with_pose>
     </link>
-    <xacro:laser_sensor parent="${roomblock_link}" visualize="$(arg visualize)"/>
+    <xacro:laser_sensor parent="${roomblock_link}" visualize="${visualize}" gpu="${gpu}"/>
     <xacro:camera_sensor parent="${roomblock_link}"/>
     <xacro:roomblock_gazebo link_name="${roomblock_link}"/>

File: ca_description/urdf/sensors/laser_sensor.xacro (robot description, xacro)
@@ -2,5 +2,5 @@
 <robot xmlns:xacro="http://ros.org/wiki/xacro">
   <xacro:include filename="$(find ca_description)/urdf/sensors/laser_sensor_gazebo.xacro"/>
-  <xacro:macro name="laser_sensor" params="parent visualize:=false">
+  <xacro:macro name="laser_sensor" params="parent visualize:=false gpu:=false">
     <xacro:property name="parent_link" value="${parent}"/>
     <xacro:property name="laser_link" value="laser_link"/>
@@ -18,5 +18,5 @@
     <link name="${laser_link}"/>
     <!-- Gazebo plugin -->
-    <xacro:laser_sensor_gazebo link_name="${laser_link}" visualize="$(arg visualize)"/>
+    <xacro:laser_sensor_gazebo link_name="${laser_link}" visualize="${visualize}" gpu="${gpu}"/>
   </xacro:macro>
 </robot>

File: ca_description/urdf/sensors/laser_sensor_gazebo.xacro (robot description, xacro)
@@ -1,5 +1,5 @@
 <?xml version="1.0"?>
 <robot xmlns:xacro="http://ros.org/wiki/xacro">
-<xacro:macro name="laser_sensor_gazebo" params="link_name visualize:=false">
+<xacro:macro name="laser_sensor_gazebo" params="link_name visualize:=false gpu:=false">
   <xacro:property name="rplidar_a2_rate_hz" value="10"/>
   <xacro:property name="rplidar_a2_min_range_m" value="0.15"/>
@@ -11,7 +11,15 @@
   <xacro:property name="laser_link" value="${link_name}"/>
   <xacro:property name="topic_name" value="laser/scan"/>
+  <xacro:if value="${gpu}">
+    <xacro:property name="ray_type" value="gpu_ray"/>
+    <xacro:property name="ray_plugin" value="libgazebo_ros_gpu_laser.so"/>
+  </xacro:if>
+  <xacro:unless value="${gpu}">
+    <xacro:property name="ray_type" value="ray"/>
+    <xacro:property name="ray_plugin" value="libgazebo_ros_laser.so"/>
+  </xacro:unless>
   <gazebo reference="${link_name}">
     <material>Gazebo/Black</material>
-    <sensor type="ray" name="rplidar_sensor">
+    <sensor type="${ray_type}" name="rplidar_sensor">
       <pose>0 0 0 0 0 0</pose>
       <visualize>${visualize}</visualize>
@@ -41,5 +49,5 @@
         </noise>
       </ray>
-      <plugin name="gazebo_ros_rplidar_controller" filename="libgazebo_ros_laser.so">
+      <plugin name="gazebo_ros_rplidar_controller" filename="${ray_plugin}">
         <topicName>${topic_name}</topicName>
         <frameName>${link_name}</frameName>
