Commit message: Add GPU flag

File: ca_description/urdf/create_2.urdf.xacro (robot description, xacro)
@@ -3,5 +3,5 @@
   <xacro:include filename="$(find ca_description)/urdf/create_base.urdf.xacro"/>
   <xacro:include filename="$(find ca_description)/urdf/roomblock.urdf.xacro"/>
-  <xacro:create_base wheel_separation="0.235" base_diameter="0.3485" visualize="$(arg visualize)">
+  <xacro:create_base wheel_separation="0.235" base_diameter="0.3485" visualize="$(arg visualize)" gpu="$(arg gpu)">
     <mesh filename="package://ca_description/meshes/create_2.dae" />
   </xacro:create_base>

File: ca_description/urdf/create_base.xacro (robot description, xacro)
@@ -1,5 +1,5 @@
 <?xml version="1.0" ?>
 <robot xmlns:xacro="http://ros.org/wiki/xacro">
-  <xacro:macro name="create_base" params="wheel_separation wheel_radius wheel_width base_diameter *mesh visualize:=false">
+  <xacro:macro name="create_base" params="wheel_separation wheel_radius wheel_width base_diameter *mesh visualize:=false gpu:=false">
     <xacro:include filename="$(find ca_description)/urdf/create_base_gazebo.xacro"/>
     <xacro:include filename="$(find ca_description)/urdf/create_caster_wheel.xacro"/>
@@ -33,6 +33,6 @@
       </collision>
     </link>
-    <xacro:wall_sensor visualize="${visualize}"/>
-    <xacro:cliff_sensors visualize="${visualize}"/>
+    <xacro:wall_sensor visualize="${visualize}" gpu="${gpu}"/>
+    <xacro:cliff_sensors visualize="${visualize}" gpu="${gpu}"/>
     <xacro:imu_sensor name="imu">
       <origin xyz="0 -0.04 0.13" rpy="0 0 0"/>

File: ca_description/urdf/sensors/cliff_sensors.xacro (robot description, xacro)
@@ -1,5 +1,5 @@
 <?xml version="1.0" ?>
 <robot xmlns:xacro="http://ros.org/wiki/xacro">
-<xacro:macro name="cliff_sensors" params="visualize:=false">
+<xacro:macro name="cliff_sensors" params="visualize:=false gpu:=false">
   <xacro:include filename="$(find ca_description)/urdf/common_properties.xacro"/>
   <xacro:include filename="$(find ca_description)/urdf/sensors/cliff_sensors_gazebo.xacro"/>
@@ -41,5 +41,5 @@
     <xacro:dummy_inertia/>
   </link>
-  <xacro:sim_create_cliff_sensors visualize="${visualize}"/>
+  <xacro:sim_create_cliff_sensors visualize="${visualize}" gpu="${gpu}"/>
 </xacro:macro>
 </robot>

File: ca_description/urdf/sensors/cliff_sensors_gazebo.xacro (robot description, xacro)
@@ -1,10 +1,19 @@
 <?xml version="1.0" ?>
 <robot xmlns:xacro="http://ros.org/wiki/xacro">
-<xacro:macro name="sim_create_cliff_sensors" params="visualize:=false">
+<xacro:macro name="sim_create_cliff_sensors" params="visualize:=false gpu:=false">
   <xacro:property name="min_range_m" value="0.01"/>
   <xacro:property name="max_range_m" value="0.04"/>
   <xacro:property name="rate_hz" value="20.0"/>
+  <!-- Use GPU lasers or not -->
+  <xacro:if value="${gpu}">
+    <xacro:property name="ray_type" value="gpu_ray"/>
+    <xacro:property name="ray_plugin" value="libgazebo_ros_gpu_laser.so"/>
+  </xacro:if>
+  <xacro:unless value="${gpu}">
+    <xacro:property name="ray_type" value="ray"/>
+    <xacro:property name="ray_plugin" value="libgazebo_ros_laser.so"/>
+  </xacro:unless>
   <gazebo reference="${name_side_left}_cliff_sensor_link">
-    <sensor type="ray" name="${name_side_left}_cliff_sensor">
+    <sensor type="${ray_type}" name="${name_side_left}_cliff_sensor">
       <always_on>true</always_on>
       <update_rate>${rate_hz}</update_rate>
@@ -26,5 +35,5 @@
         </range>
       </ray>
-      <plugin name="gazebo_ros_${name_side_left}_cliff_sensor" filename="libgazebo_ros_laser.so">
+      <plugin name="gazebo_ros_${name_side_left}_cliff_sensor" filename="${ray_plugin}">
         <topicName>${name_side_left}_cliff_sensor/scan</topicName>
         <frameName>${name_side_left}_cliff_sensor_link</frameName>
@@ -33,5 +42,5 @@
   </gazebo>
   <gazebo reference="${name_side_right}_cliff_sensor_link">
-    <sensor type="ray" name="${name_side_right}_cliff_sensor">
+    <sensor type="${ray_type}" name="${name_side_right}_cliff_sensor">
       <always_on>true</always_on>
       <update_rate>${rate_hz}</update_rate>
@@ -53,5 +62,5 @@
         </range>
       </ray>
-      <plugin name="gazebo_ros_${name_side_right}_cliff_sensor" filename="libgazebo_ros_laser.so">
+      <plugin name="gazebo_ros_${name_side_right}_cliff_sensor" filename="${ray_plugin}">
         <topicName>${name_side_right}_cliff_sensor/scan</topicName>
         <frameName>${name_side_right}_cliff_sensor_link</frameName>
@@ -60,5 +69,5 @@
   </gazebo>
   <gazebo reference="${name_front_left}_cliff_sensor_link">
-    <sensor type="ray" name="${name_front_left}_cliff_sensor">
+    <sensor type="${ray_type}" name="${name_front_left}_cliff_sensor">
       <always_on>true</always_on>
       <update_rate>${rate_hz}</update_rate>
@@ -80,5 +89,5 @@
         </range>
       </ray>
-      <plugin name="gazebo_ros_${name_front_left}_cliff_sensor" filename="libgazebo_ros_laser.so">
+      <plugin name="gazebo_ros_${name_front_left}_cliff_sensor" filename="${ray_plugin}">
         <topicName>${name_front_left}_cliff_sensor/scan</topicName>
         <frameName>${name_front_left}_cliff_sensor</frameName>
@@ -87,5 +96,5 @@
   </gazebo>
   <gazebo reference="${name_front_right}_cliff_sensor_link">
-    <sensor type="ray" name="${name_front_right}_cliff_sensor">
+    <sensor type="${ray_type}" name="${name_front_right}_cliff_sensor">
       <always_on>true</always_on>
       <update_rate>${rate_hz}</update_rate>
@@ -107,5 +116,5 @@
         </range>
       </ray>
-      <plugin name="gazebo_ros_${name_front_right}_cliff_sensor" filename="libgazebo_ros_laser.so">
+      <plugin name="gazebo_ros_${name_front_right}_cliff_sensor" filename="${ray_plugin}">
         <topicName>${name_front_right}_cliff_sensor/scan</topicName>
         <frameName>${name_front_right}_cliff_sensor</frameName>

File: ca_description/urdf/sensors/laser_sensor_gazebo.xacro (robot description, xacro)
@@ -11,4 +11,5 @@
   <xacro:property name="laser_link" value="${link_name}"/>
   <xacro:property name="topic_name" value="laser/scan"/>
+  <!-- Use GPU lasers or not -->
   <xacro:if value="${gpu}">
     <xacro:property name="ray_type" value="gpu_ray"/>

File: ca_description/urdf/sensors/wall_sensor.xacro (robot description, xacro)
@@ -1,5 +1,5 @@
 <?xml version="1.0" ?>
 <robot xmlns:xacro="http://ros.org/wiki/xacro">
-<xacro:macro name="wall_sensor" params="visualize:=false">
+<xacro:macro name="wall_sensor" params="visualize:=false gpu:=false">
   <xacro:include filename="$(find ca_description)/urdf/common_properties.xacro"/>
   <xacro:include filename="$(find ca_description)/urdf/sensors/wall_sensor_gazebo.xacro"/>
@@ -19,5 +19,5 @@
     <xacro:dummy_inertia/>
   </link>
-  <xacro:sim_create_wall_sensor visualize="${visualize}"/>
+  <xacro:sim_create_wall_sensor visualize="${visualize}" gpu="${gpu}"/>
 </xacro:macro>
 </robot>

File: ca_description/urdf/sensors/wall_sensor_gazebo.xacro (robot description, xacro)
@@ -1,11 +1,20 @@
 <?xml version="1.0" ?>
 <robot xmlns:xacro="http://ros.org/wiki/xacro">
-<xacro:macro name="sim_create_wall_sensor" params="visualize:=false">
+<xacro:macro name="sim_create_wall_sensor" params="visualize:=false gpu:=false">
   <xacro:property name="link_name" value="wall_sensor_link"/>
   <xacro:property name="rate_hz" value="20.0"/>
   <xacro:property name="min_range_m" value="0.0160"/>
   <xacro:property name="max_range_m" value="0.04"/>
+  <!-- Use GPU lasers or not -->
+  <xacro:if value="${gpu}">
+    <xacro:property name="ray_type" value="gpu_ray"/>
+    <xacro:property name="ray_plugin" value="libgazebo_ros_gpu_laser.so"/>
+  </xacro:if>
+  <xacro:unless value="${gpu}">
+    <xacro:property name="ray_type" value="ray"/>
+    <xacro:property name="ray_plugin" value="libgazebo_ros_laser.so"/>
+  </xacro:unless>
   <gazebo reference="${link_name}">
-    <sensor type="ray" name="wall_sensor">
+    <sensor type="${ray_type}" name="wall_sensor">
       <always_on>true</always_on>
       <update_rate>${rate_hz}</update_rate>
@@ -27,5 +36,5 @@
         </range>
       </ray>
-      <plugin name="gazebo_ros_wall_sensor" filename="libgazebo_ros_laser.so">
+      <plugin name="gazebo_ros_wall_sensor" filename="${ray_plugin}">
         <topicName>/wall_sensor/scan</topicName>
         <frameName>${link_name}</frameName>
